File: echo-chan.kicad_pcb (KiCad board)
At the start: 2 copper layers, 110.5 x 87 mm, 56 parts, among them J1 SJ1-3533NS, J2 USB_B, SW1 SW_Push, T1 Transformer_1P_1S, U1 JAMMA, U2 JAMMA, U3 AT90USB1286, U4 HD15, U5 AD8054, Y1 16MHz

Commit message: [PCB] Tentative layout complete
Parts:
- removed D1: LED, footprints:LED_0603_1608Metric
- removed G***: segv, footprints:segv
- removed G***: head, footprints:head
- removed R18, R19, R20, R21, R22, R23, R24, R25, R26, R27, R29, R30, R31, R32, R33: 1K, footprints:R_0805_2012Metric
- removed R37, R38, R39: 220, footprints:R_0805_2012Metric
- removed U5: AD8054, footprints:AD8054ARZ-REEL7
- added C10: 100nF, Capacitor_SMD:C_0805_2012Metric, F.Cu at (141.4, 70.2)
- added C11: 10pF, Capacitor_SMD:C_0805_2012Metric, F.Cu at (138.8, 81.9)
- added C12: 100nF, Capacitor_SMD:C_0805_2012Metric, F.Cu at (141.4, 72.2)
- added C13: 100nF, Capacitor_SMD:C_0805_2012Metric, F.Cu at (141.4, 74.2)
- added C14: 100nF, Capacitor_SMD:C_0805_2012Metric, F.Cu at (154.2, 73.9)
- added C15: 490uF, Capacitor_THT:CP_Radial_D8.0mm_P3.50mm, F.Cu at (166.2, 64.6)
- added C16: 100nF, Capacitor_SMD:C_0805_2012Metric, F.Cu at (162.2, 64.6)
- added C17: 490uF, Capacitor_THT:CP_Radial_D8.0mm_P3.50mm, F.Cu at (166.2, 73.5)
- added C18: 100nF, Capacitor_SMD:C_0805_2012Metric, F.Cu at (162.2, 73.5)
- added C19: 490uF, Capacitor_THT:CP_Radial_D8.0mm_P3.50mm, F.Cu at (166.2, 82.5)
- added C20: 100nF, Capacitor_SMD:C_0805_2012Metric, F.Cu at (162.2, 82.5)
- added C21: 490uF, Capacitor_THT:CP_Radial_D8.0mm_P3.50mm, F.Cu at (166.2, 91.4)
- added C22: 100nF, Capacitor_SMD:C_0805_2012Metric, F.Cu at (162.2, 91.4)
- added R15: 75, Resistor_SMD:R_0805_2012Metric, F.Cu at (154.2, 68.0)
- added R16: 75, Resistor_SMD:R_0805_2012Metric, F.Cu at (154.2, 70.0)
- added U6: THS7374, Package_SO:TSSOP-14_4.4x5mm_P0.65mm, F.Cu at (147.8, 72.2)
- C1, C2: value 1uF -> 100nF; footprint footprints:C_0603_1608Metric -> Capacitor_SMD:C_0805_2012Metric
- C3: value 100nF -> 10pF; footprint footprints:C_0603_1608Metric -> Capacitor_SMD:C_0805_2012Metric
- C4, C5: value 10pF -> 100nF; footprint footprints:C_0603_1608Metric -> Capacitor_SMD:C_0805_2012Metric
- C6: value 4.7uf -> 100nF; footprint footprints:C_1206_3216Metric_Pad1.42x1.75mm_HandSolder -> Capacitor_SMD:C_0805_2012Metric
- C7, C8: value 100nF -> 1uF; footprint footprints:C_0603_1608Metric -> Capacitor_SMD:C_0805_2012Metric
- C9: value 100nf -> 100nF; footprint footprints:C_0603_1608Metric -> Capacitor_SMD:C_0805_2012Metric
- J2: footprint footprints:USB_B_OST_USB-B1HSxx_Horizontal -> Connector_USB:USB_B_OST_USB-B1HSxx_Horizontal
- R1, R2, R3, R4, R40, R5, R6, R7, R8, R9: footprint footprints:R_0805_2012Metric -> Resistor_SMD:R_0805_2012Metric
- R10, R11, R12, R13: value 1K -> 390; footprint footprints:R_0805_2012Metric -> Resistor_SMD:R_0805_2012Metric
- R14, R17: value 1K -> 75; footprint footprints:R_0805_2012Metric -> Resistor_SMD:R_0805_2012Metric
- SW1: footprint footprints:BUTTON -> Button_Switch_THT:SW_PUSH_6mm
- U3: footprint footprints:TQFP-64_14x14mm_P0.8mm -> Package_QFP:TQFP-64_14x14mm_P0.8mm
- U4: footprint footprints:DSUB-15-HD_Female_Horizontal_P2.29x2.54mm_EdgePinOffset9.40mm -> echo-chan:DSUB-15-HD_Female_Horizontal_P2.29x2.54mm_EdgePinOffset9.40mm_anchors
- Y1: footprint footprints:Crystal_SMD_SeikoEpson_FA238-4Pin_3.2x2.5mm -> Crystal:Crystal_HC49-4H_Vertical
- moved C6 52.2 mm to (141.4, 68.1), turned to 0 degrees
- moved SW1 43.3 mm to (167.5, 112.2), turned to 90 degrees
- moved R6 38.2 mm to (135.0, 64.5), turned to 90 degrees
- moved R7 35.4 mm to (136.9, 64.5), turned to 90 degrees
- moved R14 34.1 mm to (154.2, 66.0), turned to 180 degrees
- moved C4 33.6 mm to (153.4, 107.4), turned to -90 degrees
- moved C5 31.9 mm to (151.2, 107.4)
- moved R8 30.8 mm to (138.9, 64.5), turned to 90 degrees
- moved R10 30.7 mm to (134.7, 68.1), turned to 180 degrees
- moved R11 29.5 mm to (134.7, 70.1), turned to 180 degrees
- moved R12 28.8 mm to (134.7, 72.2), turned to 180 degrees
- moved R17 28.8 mm to (154.2, 71.9), turned to 180 degrees
- moved R9 28.0 mm to (140.9, 64.5), turned to 90 degrees
- moved C2 26.7 mm to (143.0, 107.4), turned to -90 degrees
- moved C9 25.5 mm to (156.8, 96.3), turned to 180 degrees
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Connections:
- net Net-(R30-Pad2) renamed SERVICE
- net Net-(R31-Pad2) renamed TEST
- net Net-(R32-Pad2) renamed P1_B5
- net Net-(R33-Pad2) renamed P2_B5
- net Net-(R4-Pad1) renamed SPEAKER+
- net Net-(R40-Pad1) renamed SPEAKER-
- net Net-(U1-Pad14) renamed VIDEO_GND
- net Net-(U1-Pad8) renamed COIN_COUNT_1
- net Net-(U1-Pad9) renamed COIN_LOCK_1
- net Net-(U1-PadJ) renamed COIN_COUNT_2
- net Net-(U1-PadK) renamed COIN_LOCK_2
- net Net-(U1-PadS) renamed TILT
- C1 pad 1: +5V -> VBUS
- C2 pad 1: Net-(C2-Pad1) -> VBUS
- C3 pad 1: Net-(C3-Pad1) -> Net-(U3-XTAL2)
- C4 pad 1: Net-(C4-Pad1) -> VBUS
- C5 pad 1: Net-(C5-Pad1) -> GND
- C5 pad 2: GND -> Net-(U3-AREF)
- C6 pad 1: +5V -> Net-(C6-Pad1)
- C6 pad 2: GND -> Net-(U6-CH1_IN)
- C7 pad 1: +5V -> VBUS
- C8 pad 2: +5V -> Net-(U3-UCap)
- C9 pad 2: +5V -> VBUS
- J2 pad 1: +5V -> VBUS
- J2 pad 2: /USB-R_D- -> Net-(J2-D-)
- J2 pad 3: /USB-R_D+ -> Net-(J2-D+)
- R1 pad 1: /R-MCU_D- -> USB+
- R1 pad 2: /USB-R_D- -> Net-(J2-D+)
- R10 pad 1: Net-(R10-Pad1) -> Net-(C6-Pad1)
- R10 pad 2: Net-(R10-Pad2) -> GND
- R11 pad 1: Net-(R11-Pad1) -> Net-(C10-Pad1)
- R11 pad 2: Net-(R11-Pad2) -> GND
- R12 pad 1: Net-(R12-Pad1) -> Net-(C12-Pad1)
- R12 pad 2: Net-(R12-Pad2) -> GND
- R13 pad 1: Net-(R13-Pad1) -> Net-(C13-Pad1)
- R13 pad 2: Net-(R13-Pad2) -> GND
- R14 pad 1: Net-(R14-Pad1) -> Net-(C15-Pad1)
- R14 pad 2: Net-(R14-Pad2) -> Net-(U6-CH1_OUT)
- R17 pad 1: Net-(R17-Pad1) -> Net-(C21-Pad1)
- R17 pad 2: Net-(R17-Pad2) -> Net-(U6-CH4_OUT)
- R2 pad 1: /R-MCU_D+ -> USB-
- R2 pad 2: /USB-R_D+ -> Net-(J2-D-)
- R3 pad 1: Net-(R3-Pad1) -> GND
- R3 pad 2: GND -> Net-(U3-PE2)
- R6 pad 1: Net-(R6-Pad1) -> Net-(C6-Pad1)
- R6 pad 2: Net-(R6-Pad2) -> VIDEO_RED
- R7 pad 1: Net-(R7-Pad1) -> Net-(C10-Pad1)
- R7 pad 2: Net-(R7-Pad2) -> VIDEO_GREEN
- R8 pad 1: Net-(R8-Pad1) -> Net-(C12-Pad1)
- R8 pad 2: Net-(R8-Pad2) -> VIDEO_BLUE
- R9 pad 1: Net-(R9-Pad1) -> Net-(C13-Pad1)
- R9 pad 2: Net-(R9-Pad2) -> VIDEO_SYNC
- T1 pad SH: GND -> (no net)
- U1 pad 11: Net-(U1-Pad11) -> unconnected-(U1-NC-Pad11)
- U1 pad 12: Net-(U1-Pad12) -> VIDEO_RED
- U1 pad 13: Net-(U1-Pad13) -> VIDEO_BLUE
- U1 pad 16: Net-(R26-Pad2) -> COIN_1
- U1 pad 17: Net-(R24-Pad2) -> P1_START
- U1 pad 18: Net-(R6-Pad2) -> P1_UP
- U1 pad 19: Net-(R7-Pad2) -> P1_DOWN
- U1 pad 20: Net-(R8-Pad2) -> P1_LEFT
- U1 pad 21: Net-(R9-Pad2) -> P1_RIGHT
- U1 pad 22: Net-(R14-Pad2) -> P1_B1
- U1 pad 23: Net-(R17-Pad2) -> P1_B2
- U1 pad 24: Net-(R18-Pad2) -> P1_B3
- U1 pad 25: Net-(R19-Pad2) -> P1_B4
- U1 pad 7: Net-(U1-Pad7) -> unconnected-(U1-KEY-Pad7)
- U1 pad H: Net-(U1-PadH) -> unconnected-(U1-KEY-PadH)
- U1 pad M: Net-(U1-PadM) -> unconnected-(U1-NC-PadM)
- U1 pad N: Net-(U1-PadN) -> VIDEO_GREEN
- U1 pad P: Net-(U1-PadP) -> VIDEO_SYNC
- U1 pad T: Net-(R27-Pad2) -> COIN_2
- U1 pad U: Net-(R25-Pad2) -> P2_START
- U1 pad V: Net-(R10-Pad2) -> P2_UP
- U1 pad W: Net-(R11-Pad2) -> P2_DOWN
- U1 pad X: Net-(R12-Pad2) -> P2_LEFT
- U1 pad Y: Net-(R13-Pad2) -> P2_RIGHT
- U1 pad Z: Net-(R20-Pad2) -> P2_B1
- U1 pad a: Net-(R21-Pad2) -> P2_B2
- U1 pad b: Net-(R22-Pad2) -> P2_B3
- U1 pad c: Net-(R23-Pad2) -> P2_B4
- U2 pad 11: Net-(U1-Pad11) -> unconnected-(U2-NC-Pad11)
- U2 pad 12: Net-(U1-Pad12) -> VIDEO_RED
- U2 pad 13: Net-(U1-Pad13) -> VIDEO_BLUE
- U2 pad 16: Net-(R26-Pad2) -> COIN_1
- U2 pad 17: Net-(R24-Pad2) -> P1_START
- U2 pad 18: Net-(R6-Pad2) -> P1_UP
- U2 pad 19: Net-(R7-Pad2) -> P1_DOWN
- U2 pad 20: Net-(R8-Pad2) -> P1_LEFT
- U2 pad 21: Net-(R9-Pad2) -> P1_RIGHT
- U2 pad 22: Net-(R14-Pad2) -> P1_B1
- U2 pad 23: Net-(R17-Pad2) -> P1_B2
- U2 pad 24: Net-(R18-Pad2) -> P1_B3
- U2 pad 25: Net-(R19-Pad2) -> P1_B4
- U2 pad 7: Net-(U2-Pad7) -> unconnected-(U2-KEY-Pad7)
- U2 pad H: Net-(U2-PadH) -> unconnected-(U2-KEY-PadH)
- U2 pad M: Net-(U1-PadM) -> unconnected-(U2-NC-PadM)
- U2 pad N: Net-(U1-PadN) -> VIDEO_GREEN
- U2 pad P: Net-(U1-PadP) -> VIDEO_SYNC
- U2 pad T: Net-(R27-Pad2) -> COIN_2
- U2 pad U: Net-(R25-Pad2) -> P2_START
- U2 pad V: Net-(R10-Pad2) -> P2_UP
- U2 pad W: Net-(R11-Pad2) -> P2_DOWN
- U2 pad X: Net-(R12-Pad2) -> P2_LEFT
- U2 pad Y: Net-(R13-Pad2) -> P2_RIGHT
- U2 pad Z: Net-(R20-Pad2) -> P2_B1
- U2 pad a: Net-(R21-Pad2) -> P2_B2
- U2 pad b: Net-(R22-Pad2) -> P2_B3
- U2 pad c: Net-(R23-Pad2) -> P2_B4
- U3 pad 1: Net-(U3-Pad1) -> P1_START
- U3 pad 10: Net-(R6-Pad1) -> P1_DOWN
- U3 pad 11: Net-(R7-Pad1) -> P1_LEFT
- U3 pad 12: Net-(R8-Pad1) -> P1_RIGHT
- U3 pad 13: Net-(R9-Pad1) -> P2_UP
- U3 pad 14: Net-(R10-Pad1) -> P2_DOWN
- U3 pad 15: Net-(R11-Pad1) -> P2_LEFT
- U3 pad 16: Net-(R12-Pad1) -> P2_RIGHT
- U3 pad 17: Net-(R13-Pad1) -> unconnected-(U3-PB7-Pad17)
- U3 pad 18: Net-(U3-Pad18) -> unconnected-(U3-PE4-Pad18)
- U3 pad 19: Net-(U3-Pad19) -> unconnected-(U3-PE5-Pad19)
- U3 pad 2: Net-(U3-Pad2) -> P2_START
- U3 pad 21: +5V -> VBUS
- U3 pad 23: Net-(C4-Pad1) -> Net-(U3-XTAL2)
- U3 pad 24: Net-(C5-Pad1) -> Net-(U3-XTAL1)
- U3 pad 25: Net-(U3-Pad25) -> unconnected-(U3-PD0-Pad25)
- U3 pad 26: Net-(U3-Pad26) -> unconnected-(U3-PD1-Pad26)
- U3 pad 27: Net-(U3-Pad27) -> unconnected-(U3-PD2-Pad27)
- U3 pad 28: Net-(U3-Pad28) -> unconnected-(U3-PD3-Pad28)
- U3 pad 29: Net-(U3-Pad29) -> unconnected-(U3-PD4-Pad29)
- U3 pad 3: +5V -> VBUS
- U3 pad 30: Net-(U3-Pad30) -> unconnected-(U3-PD5-Pad30)
- U3 pad 31: Net-(D1-Pad2) -> unconnected-(U3-PD6-Pad31)
- U3 pad 32: Net-(U3-Pad32) -> unconnected-(U3-PD7-Pad32)
- U3 pad 33: Net-(U3-Pad33) -> unconnected-(U3-PE0-Pad33)
- U3 pad 34: Net-(U3-Pad34) -> unconnected-(U3-PE1-Pad34)
- U3 pad 35: Net-(R24-Pad1) -> unconnected-(U3-PC0-Pad35)
- U3 pad 36: Net-(R25-Pad1) -> unconnected-(U3-PC1-Pad36)
- U3 pad 37: Net-(R26-Pad1) -> unconnected-(U3-PC2-Pad37)
- U3 pad 38: Net-(R27-Pad1) -> unconnected-(U3-PC3-Pad38)
- U3 pad 39: Net-(R30-Pad1) -> unconnected-(U3-PC4-Pad39)
- U3 pad 4: /R-MCU_D- -> USB-
- U3 pad 40: Net-(R31-Pad1) -> unconnected-(U3-PC5-Pad40)
- U3 pad 41: Net-(R32-Pad1) -> unconnected-(U3-PC6-Pad41)
- U3 pad 42: Net-(R33-Pad1) -> unconnected-(U3-PC7-Pad42)
- U3 pad 43: Net-(R3-Pad1) -> Net-(U3-PE2)
- U3 pad 44: Net-(R23-Pad1) -> unconnected-(U3-PA7-Pad44)
- U3 pad 45: Net-(R22-Pad1) -> unconnected-(U3-PA6-Pad45)
- U3 pad 46: Net-(R21-Pad1) -> unconnected-(U3-PA5-Pad46)
- U3 pad 47: Net-(R20-Pad1) -> unconnected-(U3-PA4-Pad47)
- U3 pad 48: Net-(R19-Pad1) -> unconnected-(U3-PA3-Pad48)
- U3 pad 49: Net-(R18-Pad1) -> unconnected-(U3-PA2-Pad49)
- U3 pad 5: /R-MCU_D+ -> USB+
- U3 pad 50: Net-(R17-Pad1) -> COIN_1
- U3 pad 51: Net-(R14-Pad1) -> COIN_2
- U3 pad 52: +5V -> VBUS
- U3 pad 54: Net-(U3-Pad54) -> P2_B4
- U3 pad 55: Net-(U3-Pad55) -> P2_B3
- U3 pad 56: Net-(U3-Pad56) -> P2_B2
- U3 pad 57: Net-(U3-Pad57) -> P2_B1
- U3 pad 58: Net-(U3-Pad58) -> P1_B4
- U3 pad 59: Net-(U3-Pad59) -> P1_B3
- U3 pad 60: Net-(U3-Pad60) -> P1_B2
- U3 pad 61: Net-(U3-Pad61) -> P1_B1
- U3 pad 62: Net-(C3-Pad1) -> Net-(U3-AREF)
- U3 pad 63: Net-(U3-Pad63) -> GND
- U3 pad 64: +5V -> VBUS
- U3 pad 7: Net-(C2-Pad1) -> Net-(U3-UCap)
- U3 pad 8: +5V -> VBUS
- U3 pad 9: Net-(U3-Pad9) -> P1_UP
- U4 pad 1: Net-(R37-Pad2) -> HD15_RED
- U4 pad 11: Net-(U4-Pad11) -> unconnected-(U4-ID0-Pad11)
- U4 pad 12: Net-(U4-Pad12) -> unconnected-(U4-SDA-Pad12)
- U4 pad 13: Net-(U1-PadP) -> HD15_SYNC
- U4 pad 14: Net-(U4-Pad14) -> unconnected-(U4-VSYNC-Pad14)
- U4 pad 15: Net-(U4-Pad15) -> unconnected-(U4-SCL-Pad15)
- U4 pad 2: Net-(R38-Pad2) -> HD15_BLUE
- U4 pad 3: Net-(R39-Pad2) -> HD15_BLUE
- U4 pad 4: Net-(U4-Pad4) -> unconnected-(U4-RES-Pad4)
- U4 pad 9: Net-(U4-Pad9) -> unconnected-(U4-KEY-Pad9)
- Y1 pad 1: Net-(C4-Pad1) -> Net-(U3-XTAL2)
- Y1 pad 2: Net-(C5-Pad1) -> Net-(U3-XTAL1)
Routing:
- net GND: track 239.5 -> 0.00 mm, vias 9 -> 0
- net +5V: track 221.1 -> 0.00 mm, vias 10 -> 0
- net Net-(R26-Pad2): track 177.2 -> 0.00 mm, vias 5 -> 0
- net SERVICE: track 177.0 -> 0.00 mm, vias 3 -> 0
- net Net-(R24-Pad2): track 174.1 -> 0.00 mm, vias 3 -> 0
- net Net-(R25-Pad2): track 171.9 -> 0.00 mm, vias 3 -> 0
- net Net-(R27-Pad2): track 171.1 -> 0.00 mm, vias 5 -> 0
- net TEST: track 168.9 -> 0.00 mm, vias 3 -> 0
- net Net-(U1-PadP): track 164.5 -> 0.00 mm, vias 5 -> 0
- net P1_B5: track 158.9 -> 0.00 mm, vias 3 -> 0
- net VIDEO_GND: track 158.9 -> 0.00 mm, vias 5 -> 0
- net Net-(U1-PadN): track 157.9 -> 0.00 mm, vias 4 -> 0
- net Net-(U1-Pad12): track 156.7 -> 0.00 mm, vias 4 -> 0
- net P2_B5: track 150.9 -> 0.00 mm, vias 1 -> 0
- net Net-(R23-Pad2): track 141.7 -> 0.00 mm, vias 1 -> 0
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- removed copper zone on B.Cu, net +12V
- removed copper zone on F.Cu, net +12V
- removed copper zone on B.Cu, net +5V
- removed copper zone on F.Cu, net +5V
- removed copper zone on B.Cu, net -5V
- removed copper zone on F.Cu, net -5V
- removed copper zone on B.Cu, net GND
- removed copper zone on F.Cu, net GND

Commit message: checkpoint
Parts:
- moved SW1 75.3 mm to (106.9, 67.4), turned to 180 degrees
- moved R40 57.3 mm to (113.9, 65.7), turned to -90 degrees
- moved R4 54.8 mm to (115.8, 65.7), turned to -90 degrees
- moved R5 54.6 mm to (114.9, 68.4), turned to 180 degrees
- moved R2 4.61 mm to (171.1, 104.7)
- moved R3 4.60 mm to (140.2, 99.4), turned to -90 degrees
- moved C2 4.11 mm to (146.8, 108.9)
- moved C4 4.11 mm to (157.2, 108.9)
- moved C5 4.11 mm to (155.1, 108.9)
- moved C8 4.11 mm to (160.6, 99.9)
- moved U3 4.11 mm to (150.1, 98.3)
- moved C9 4.11 mm to (160.6, 97.8)
- moved C1 3.59 mm to (152.5, 87.8), turned to 90 degrees
- moved C11 3.55 mm to (142.3, 82.3)
- moved C3 3.55 mm to (156.6, 82.3)
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Connections:
- U4 pad 2: HD15_BLUE -> HD15_GREEN
Routing:
- net P2_B4: track 0.00 -> 178.7 mm, vias 0 -> 3
- net P1_LEFT: track 0.00 -> 171.9 mm, vias 0 -> 4
- net P1_B4: track 0.00 -> 169.7 mm, vias 0 -> 4
- net P2_LEFT: track 0.00 -> 169.3 mm, vias 0 -> 4
- net P2_B3: track 0.00 -> 167.2 mm, vias 0 -> 4
- net P2_B2: track 0.00 -> 166.2 mm, vias 0 -> 4
- net P1_DOWN: track 0.00 -> 163.3 mm, vias 0 -> 4
- net P1_B3: track 0.00 -> 162.4 mm, vias 0 -> 4
- net P1_RIGHT: track 0.00 -> 157.9 mm, vias 0 -> 3
- net P2_RIGHT: track 0.00 -> 157.4 mm, vias 0 -> 3
- net P2_UP: track 0.00 -> 156.6 mm, vias 0 -> 3
- net P2_DOWN: track 0.00 -> 155.5 mm, vias 0 -> 4
- net P1_UP: track 0.00 -> 152.2 mm, vias 0 -> 4
- net P2_B1: track 0.00 -> 151.2 mm, vias 0 -> 4
- net P1_B1: track 0.00 -> 150.7 mm, vias 0 -> 4
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Other:
- board size 110.5 x 87 mm -> 113.5 x 87 mm

Commit message: checkpoint
Parts:
- moved SW1 6.76 mm to (112.3, 71.5), turned to -90 degrees
- moved R1 2.73 mm to (168.4, 102.7)
- moved R2 2.73 mm to (168.4, 104.9)
- moved C7 2.17 mm to (172.7, 99.1), turned to 90 degrees
- moved C11 1.09 mm to (142.3, 81.2)
- moved C3 1.09 mm to (156.6, 81.2)
- moved Y1 1.09 mm to (151.9, 81.2)
- moved C8 0.95 mm to (161.5, 99.5)
- moved C9 0.92 mm to (161.5, 97.5)
- moved C2 0.85 mm to (146.8, 109.7)
- moved C1 0.58 mm to (152.8, 87.3)
Connections:
- net Net-(J2-D+) renamed USB_PORT+
- net Net-(J2-D-) renamed USB_PORT-
- net USB+ renamed USB_MCU+
- net USB- renamed USB_MCU-
Routing:
- net Net-(T1-SA): track 0.00 -> 112.5 mm
- net Net-(T1-SB): track 0.00 -> 101.8 mm
- net Net-(U3-RESET): track 0.00 -> 66.8 mm, vias 0 -> 1
- net VIDEO_GND: track 86.7 -> 152.2 mm
- net VBUS: track 8.79 -> 68.1 mm, vias 0 -> 2
- net HD15_SYNC: track 8.29 -> 31.9 mm
- net HD15_RED: track 8.29 -> 20.6 mm
- net HD15_BLUE: track 8.29 -> 20.5 mm
- net USB_PORT+: track 0.00 -> 11.1 mm
- net GND: track 0.00 -> 9.62 mm, vias 0 -> 6
- net USB_PORT-: track 0.00 -> 9.05 mm
- net HD15_GREEN: track 8.29 -> 16.6 mm
- net Net-(U3-XTAL2): track 13.7 -> 17.7 mm
- net USB_MCU+: track 13.8 -> 10.4 mm
- net USB_MCU-: track 13.6 -> 11.1 mm
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- added copper zone on B.Cu, net +12V
- added copper zone on F.Cu, net +12V
- added copper zone on B.Cu, net +5V
- added copper zone on F.Cu, net +5V
- added copper zone on B.Cu, net -5V
- added copper zone on F.Cu, net -5V
- added copper zone on B.Cu, net GND
- added copper zone on F.Cu, net GND

Commit message: checkpoint
Parts:
- moved C2 2.10 mm to (144.8, 109.4), turned to 180 degrees
Routing:
- net +5V: track 3.46 -> 98.1 mm, vias 0 -> 3
- net GND: track 9.62 -> 27.7 mm, vias 6 -> 28
- net P2_LEFT: track 168.5 -> 162.5 mm
- net P1_START: track 146.8 -> 143.5 mm
- net P2_START: track 147.8 -> 151.0 mm
- net P1_LEFT: track 171.9 -> 168.9 mm
- net P1_DOWN: track 163.6 -> 160.6 mm
- net VIDEO_SYNC: track 98.7 -> 96.6 mm
- net VBUS: track 68.1 -> 70.3 mm
- net P1_UP: track 152.2 -> 153.5 mm
- net COIN_1: track 128.6 -> 129.4 mm
- net P2_UP: track 157.0 -> 156.4 mm
- net VIDEO_RED: track 98.7 -> 98.2 mm
- net P1_B2: track 147.0 -> 146.5 mm
- net -5V: vias 0 -> 1
Other:
- rule pad_to_mask_clearance: 0.2 -> 0.1

Commit message: route done
Routing:
- net GND: track 27.7 -> 84.1 mm, vias 28 -> 45
- net -5V: vias 1 -> 8
- net +5V: vias 3 -> 17
- net +12V: vias 0 -> 8
