File: echo-chan.kicad_pcb (KiCad board)
At the start: 2 copper layers, 110.5 x 87 mm, 50 parts, among them J1 SJ1-3533NS, J2 USB_B, SW1 SW_Push, T1 Transformer_1P_1S, U1 JAMMA, U2 JAMMA, U3 AT90USB1286, U4 HD15, U6 THS7374, Y1 16MHz

Commit message: [PCB] Routing done
Parts:
- moved SW1 68.6 mm to (112.3, 71.5), turned to -90 degrees
- moved R40 57.3 mm to (113.9, 65.7), turned to -90 degrees
- moved R4 54.8 mm to (115.8, 65.7), turned to -90 degrees
- moved R5 54.6 mm to (114.9, 68.4), turned to 180 degrees
- moved R2 5.53 mm to (168.4, 104.9)
- moved C8 4.86 mm to (161.5, 99.5)
- moved C9 4.85 mm to (161.5, 97.5)
- moved R3 4.60 mm to (140.2, 99.4), turned to -90 degrees
- moved C4 4.11 mm to (157.2, 108.9)
- moved C5 4.11 mm to (155.1, 108.9)
- moved U3 4.11 mm to (150.1, 98.3)
- moved C1 3.82 mm to (152.8, 87.3), turned to 90 degrees
- moved C11 3.60 mm to (142.3, 81.2)
- moved C3 3.60 mm to (156.6, 81.2)
- moved Y1 3.60 mm to (151.9, 81.2)
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Connections:
- net Net-(J2-D+) renamed USB_PORT+
- net Net-(J2-D-) renamed USB_PORT-
- net USB+ renamed USB_MCU+
- net USB- renamed USB_MCU-
- U4 pad 2: HD15_BLUE -> HD15_GREEN
Routing:
- net P2_B4: track 0.00 -> 178.7 mm, vias 0 -> 3
- net P1_B4: track 0.00 -> 169.7 mm, vias 0 -> 4
- net P1_LEFT: track 0.00 -> 168.9 mm, vias 0 -> 4
- net P2_B3: track 0.00 -> 167.2 mm, vias 0 -> 4
- net P2_B2: track 0.00 -> 166.2 mm, vias 0 -> 4
- net P2_LEFT: track 0.00 -> 162.5 mm, vias 0 -> 4
- net P1_B3: track 0.00 -> 162.4 mm, vias 0 -> 4
- net P1_DOWN: track 0.00 -> 160.6 mm, vias 0 -> 4
- net P1_RIGHT: track 0.00 -> 157.6 mm, vias 0 -> 2
- net P2_RIGHT: track 0.00 -> 157.3 mm, vias 0 -> 4
- net P2_UP: track 0.00 -> 156.4 mm, vias 0 -> 3
- net P2_DOWN: track 0.00 -> 156.1 mm, vias 0 -> 4
- net P1_UP: track 0.00 -> 153.5 mm, vias 0 -> 4
- net VIDEO_GND: track 0.00 -> 152.2 mm, vias 0 -> 2
- net P2_B1: track 0.00 -> 151.2 mm, vias 0 -> 4
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- added copper zone on B.Cu, net +12V
- added copper zone on F.Cu, net +12V
- added copper zone on B.Cu, net +5V
- added copper zone on F.Cu, net +5V
- added copper zone on B.Cu, net -5V
- added copper zone on F.Cu, net -5V
- added copper zone on B.Cu, net GND
- added copper zone on F.Cu, net GND
Other:
- board size 110.5 x 87 mm -> 113.5 x 87 mm
- rule pad_to_mask_clearance: 0.2 -> 0.1
