File: pcb/echo-chan.kicad_pcb (KiCad board)
At the start: 2 copper layers, 113.5 x 87 mm, 50 parts, among them J1 SJ1-3533NS, J2 USB_B, SW1 SW_Push, T1 Transformer_1P_1S, U1 JAMMA, U2 JAMMA, U3 AT90USB1286, U4 HD15, U6 THS7374, Y1 16MHz

Commit message: [PCB] Add silkscreen
Parts:
- added G***: LOGO, LOGO, B.Cu at (137.8, 97.5)
- added G***: LOGO, LOGO, B.Cu at (135.8, 76.8)
Other:
- board text added: "1995 - 2024"
